File: board/board.sch (KiCad schematic (older format))
At the start: 57 parts, among them J1 programmer, J2 USB_B_Micro, Q1 Q_PMOS_DSG, Q2 Q_NMOS_GSD, U1 ESP-WROOM-02, U2 RT8097AHGB, U3 RT8097AHGB, U4 NPIC6C596, U5 NPIC6C596

Commit message: Pcb close
Parts:
- removed C7: 100n, Capacitor_SMD:C_0603_1608Metric_Pad1.08x0.95mm_HandSolder, symbol Device:C_Small
- removed JP1, JP2, JP3: x, Jumper:SolderJumper-2_P1.3mm_Open_TrianglePad1.0x1.5mm, symbol Jumper:SolderJumper_2_Open
- added H1, H2: MountingHole_Pad, MountingHole:MountingHole_2.2mm_M2_ISO7380_Pad, symbol Mechanical:MountingHole_Pad
- C1, C10, C11, C12, C2, C3, C4, C5, C6, C8, C9: footprint Capacitor_SMD:C_0603_1608Metric_Pad1.08x0.95mm_HandSolder -> Capacitor_SMD:C_0603_1608Metric
- J1: footprint Connector_PinHeader_2.54mm:PinHeader_1x05_P2.54mm_Vertical -> good_things:TSM-105-01-L_SH
- J2: symbol Connector:USB_B_Micro -> board-rescue:USB_B_Micro-Connector
- U2, U3: symbol good_things:RT8097AHGB -> board-rescue:RT8097AHGB-good_things
- U4, U5: footprint Package_SO:SO-16_3.9x9.9mm_P1.27mm -> Package_SO:STC_SOP-16_3.9x9.9mm_P1.27mm; symbol good_things:NPIC6C595 -> board-rescue:NPIC6C595-good_things
Connections:
- net GND: now also H1.1, H2.1
- net led_h0: now also U4.3 (q0); no longer U4.11 (q4)
- net led_h1: now also U4.4 (q1); no longer U4.6 (q3)
- net led_h3: now also U4.13 (q6); no longer U4.4 (q1)
- net led_h4: now also U4.14 (q7); no longer U4.3 (q0)
- net led_m3: now also U4.6 (q3); no longer U4.14 (q7)
- net led_m4: now also U4.11 (q4); no longer U4.13 (q6)
- net led_s0: now also D17.1 (K), Q2.3 (D); no longer R9.2, U1.17 (IO16)
- net mcu_en: now reaches C1.1, R1.2, R2.1, U1.2 (EN)
- net 3v3_sw: now reaches L1.1, U2.3 (lx)
- net 3v3_fb: now reaches C9.2, R5.2, R6.1, U2.5 (fb)
- net vled_sw: now reaches L2.1, U3.3 (lx)
- net vled_fb: now reaches C10.2, R7.2, R8.1, U3.5 (fb)
- net shift_clk_backup: no longer names the net of U1.5 (IO13)
- net shift_data_backup: no longer names the net of U1.3 (IO14)
- net store_clk_backup renamed led_s0_ctrl
- net led_s0_ctrl: now also R9.2
- no-connect marks 9 -> 12
Other:
- moved on the sheet: C4, D1, D2, D4, D5, D7, D8

Commit message: Rev1 PCB
Parts:
- removed C1: 100n, Capacitor_SMD:C_0603_1608Metric, symbol Device:C_Small
- removed R2: 10k, Resistor_SMD:R_0603_1608Metric, symbol Device:R_Small
- removed TP1, TP2, TP3: TestPoint_2Pole, good_things:TestPoint2Pole, symbol Connector:TestPoint_2Pole
- added TP1, TP3: TestPoint, TestPoint:TestPoint_Pad_D1.5mm, symbol Connector:TestPoint
Connections:
- net +3V3: now also TP1.1
- net vled: now also TP3.1
Changed lines of the file:
@@
 NoConn ~ 1350 6150
-$Comp
-L Connector:TestPoint_2Pole TP3
-U 1 1 612CDFC5
-P 2050 5750
-F 0 "TP3" V 2004 5808 50  0000 L CNN
-F 1 "TestPoint_2Pole" V 2095 5808 50  0000 L CNN
-F 2 "good_things:TestPoint2Pole" H 2050 5750 50  0001 C CNN
-F 3 "~" H 2050 5750 50  0001 C CNN
-	1    2050 5750
-	0    1    1    0
-$EndComp
 $Comp
 L power:GND #PWR06
@@
 	1    0    0    -1
 $EndComp
-$Comp
-L power:GND #PWR09
-U 1 1 612CF450
-P 2050 5950
-F 0 "#PWR09" H 2050 5700 50  0001 C CNN
-F 1 "GND" H 2055 5777 50  0000 C CNN
-F 2 "" H 2050 5950 50  0001 C CNN
-F 3 "" H 2050 5950 50  0001 C CNN
-	1    2050 5950
-	1    0    0    -1
-$EndComp
 NoConn ~ 1750 5750
 NoConn ~ 1750 5850
 NoConn ~ 1750 5950
-Wire Wire Line
-	2050 5550 1750 5550
-Connection ~ 2050 5550
 $Comp
 L Device:C_Small C3
@@
 Wire Wire Line
 	2850 5600 2850 5550
-Wire Wire Line
-	2050 5550 2850 5550
 $Comp
 L power:GND #PWR012
@@
 Connection ~ 5700 3200
 $Comp
-L Connector:TestPoint_2Pole TP1
-U 1 1 612F4595
-P 1250 6900
-F 0 "TP1" V 1204 6958 50  0000 L CNN
-F 1 "TestPoint_2Pole" V 1295 6958 50  0000 L CNN
-F 2 "good_things:TestPoint2Pole" H 1250 6900 50  0001 C CNN
-F 3 "~" H 1250 6900 50  0001 C CNN
-	1    1250 6900
-	0    1    1    0
-$EndComp
-$Comp
-L power:GND #PWR04
-U 1 1 612F459B
-P 1250 7100
-F 0 "#PWR04" H 1250 6850 50  0001 C CNN
-F 1 "GND" H 1255 6927 50  0000 C CNN
-F 2 "" H 1250 7100 50  0001 C CNN
-F 3 "" H 1250 7100 50  0001 C CNN
-	1    1250 7100
-	1    0    0    -1
-$EndComp
-$Comp
 L power:+3V3 #PWR03
 U 1 1 612F4C8A
-P 1250 6700
-F 0 "#PWR03" H 1250 6550 50  0001 C CNN
-F 1 "+3V3" H 1265 6873 50  0000 C CNN
-F 2 "" H 1250 6700 50  0001 C CNN
-F 3 "" H 1250 6700 50  0001 C CNN
-	1    1250 6700
+P 1300 6700
+F 0 "#PWR03" H 1300 6550 50  0001 C CNN
+F 1 "+3V3" H 1315 6873 50  0000 C CNN
+F 2 "" H 1300 6700 50  0001 C CNN
+F 3 "" H 1300 6700 50  0001 C CNN
+	1    1300 6700
 	1    0    0    -1
 $EndComp
@@
 	7450 5800 7150 5800
 Connection ~ 7150 5800
-$Comp
-L Connector:TestPoint_2Pole TP2
-U 1 1 6149F2E6
-P 1950 6950
-F 0 "TP2" V 1904 7008 50  0000 L CNN
-F 1 "TestPoint_2Pole" V 1995 7008 50  0000 L CNN
-F 2 "good_things:TestPoint2Pole" H 1950 6950 50  0001 C CNN
-F 3 "~" H 1950 6950 50  0001 C CNN
-	1    1950 6950
-	0    1    1    0
-$EndComp
-$Comp
-L power:GND #PWR08
-U 1 1 6149F2EC
-P 1950 7150
-F 0 "#PWR08" H 1950 6900 50  0001 C CNN
-F 1 "GND" H 1955 6977 50  0000 C CNN
-F 2 "" H 1950 7150 50  0001 C CNN
-F 3 "" H 1950 7150 50  0001 C CNN
-	1    1950 7150
-	1    0    0    -1
-$EndComp
 Text GLabel 1950 6750 1    50   Input ~ 0
 vled
@@
 Wire Wire Line
 	2600 1150 2600 1250
-Connection ~ 1050 1450
-$Comp
-L power:GND #PWR02
-U 1 1 6121EE15
-P 1050 1450
-F 0 "#PWR02" H 1050 1200 50  0001 C CNN
-F 1 "GND" H 1055 1277 50  0000 C CNN
-F 2 "" H 1050 1450 50  0001 C CNN
-F 3 "" H 1050 1450 50  0001 C CNN
-	1    1050 1450
-	1    0    0    -1
-$EndComp
 NoConn ~ 2300 1550
 Wire Wire Line
-	1050 1450 1400 1450
-Wire Wire Line
-	1050 1200 1400 1200
-Wire Wire Line
-	1050 1250 1050 1200
-Wire Wire Line
-	1400 1200 1400 1250
-Connection ~ 1400 1200
-Wire Wire Line
 	1400 1150 1400 1200
 Wire Wire Line
 	2000 1200 1400 1200
-$Comp
-L Device:C_Small C1
-U 1 1 6121DA61
-P 1050 1350
-F 0 "C1" H 1142 1396 50  0000 L CNN
-F 1 "100n" H 1142 1305 50  0000 L CNN
-F 2 "Capacitor_SMD:C_0603_1608Metric" H 1050 1350 50  0001 C CNN
-F 3 "~" H 1050 1350 50  0001 C CNN
-	1    1050 1350
-	1    0    0    -1
-$EndComp
-$Comp
-L Device:R_Small R2
-U 1 1 6121D2A0
-P 1400 1350
-F 0 "R2" H 1459 1396 50  0000 L CNN
-F 1 "10k" H 1459 1305 50  0000 L CNN
-F 2 "Resistor_SMD:R_0603_1608Metric" H 1400 1350 50  0001 C CNN
-F 3 "~" H 1400 1350 50  0001 C CNN
-	1    1400 1350
-	1    0    0    -1
-$EndComp
 $Comp
 L Device:R_Small R1
@@
 Wire Wire Line
 	2950 7050 2950 6850
+$Comp
+L Connector:TestPoint TP3
+U 1 1 616DF0FA
+P 1950 6750
+F 0 "TP3" H 2008 6868 50  0000 L CNN
+F 1 "TestPoint" H 2008 6777 50  0000 L CNN
+F 2 "TestPoint:TestPoint_Pad_D1.5mm" H 2150 6750 50  0001 C CNN
+F 3 "~" H 2150 6750 50  0001 C CNN
+	1    1950 6750
+	-1   0    0    1
+$EndComp
+$Comp
+L Connector:TestPoint TP1
+U 1 1 616DFA07
+P 1300 6700
+F 0 "TP1" H 1358 6818 50  0000 L CNN
+F 1 "TestPoint" H 1358 6727 50  0000 L CNN
+F 2 "TestPoint:TestPoint_Pad_D1.5mm" H 1500 6700 50  0001 C CNN
+F 3 "~" H 1500 6700 50  0001 C CNN
+	1    1300 6700
+	-1   0    0    1
+$EndComp
+Wire Wire Line
+	1750 5550 2850 5550
 $EndSCHEMATC
