File: board/board.kicad_pcb (KiCad board)
At the start: 2 copper layers, 44.2 x 26 mm, 55 parts, among them J1 programmer, J2 USB_B_Micro, Q1 Q_PMOS_DSG, Q2 Q_NMOS_GSD, U1 ESP-WROOM-02, U2 RT8097AHGB, U3 RT8097AHGB, U4 NPIC6C596, U5 NPIC6C596

Commit message: Rev1 PCB
Parts:
- removed C1: 100n, Capacitor_SMD:C_0603_1608Metric
- removed R2: 10k, Resistor_SMD:R_0603_1608Metric
- removed TP2: TestPoint_2Pole, good_things:TestPoint2Pole
- R1: moved to B.Cu
- TP1, TP3: value TestPoint_2Pole -> TestPoint; footprint good_things:TestPoint2Pole -> TestPoint:TestPoint_Pad_D1.5mm
- moved TP1 38.6 mm to (68.3, 127.7), turned to 0 degrees
- moved R1 19.4 mm to (90.2, 107.8), turned to 270 degrees
- moved TP3 18.6 mm to (109.7, 130.6), turned to 0 degrees
- moved C2 1.50 mm to (91.7, 107.8)
- moved R4 1.21 mm to (103.6, 115.5)
- moved R3 1.20 mm to (69.0, 120.0)
- moved C8 0.10 mm to (68.8, 122.3)
Connections:
- TP3 pad 1: /vin_dirty -> vled
Routing:
- net GND: track 18.9 -> 33.1 mm, vias 16 -> 20
- net /rst: track 10.4 -> 13.1 mm
- net +3V3: track 13.8 -> 11.8 mm, vias 12 -> 13
- net /mcu_en: track 0.00 -> 1.59 mm
- net /led_m4: track 29.5 -> 28.8 mm
- net /led_m5: track 34.6 -> 34.1 mm
Other:
- board text added: "Binuhr tiny Rev1 2021 Anton Lööf"
- board text added: "boot"
- board text added: "gnd"
- board text added: "rst"
- board text added: "rx"
- board text added: "tx"

Commit message: Add jlc order no silk
Other:
- board text added: "JLCJLCJLCJLC"
Changed lines of the file:
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@@
   (general
     (thickness 1.6)
-    (drawings 10)
+    (drawings 11)
     (tracks 407)
     (zones 0)
@@
       (outputformat 1)
       (mirror false)
-      (drillshape 1)
+      (drillshape 0)
       (scaleselection 1)
-      (outputdirectory ""))
+      (outputdirectory "binuhr_tiny_anton_loof"))
   )
   (net 0 "")
@@
     (tags "net tie")
     (attr virtual)
-    (fp_text reference NT1 (at 4.9 6.75) (layer B.SilkS)
+    (fp_text reference NT1 (at 5.1 4.55) (layer B.SilkS)
       (effects (font (size 1 1) (thickness 0.15)) (justify mirror))
     )
@@
     )
   )
+  (gr_text JLCJLCJLCJLC (at 79.7 108.6) (layer B.SilkS)
+    (effects (font (size 1 1) (thickness 0.15)) (justify mirror))
+  )
   (gr_text "Binuhr tiny \nRev1 2021\nAnton Lööf " (at 99.6 118.8) (layer B.SilkS)
