File: board/board.kicad_pcb (KiCad board)
At the start: 2 copper layers, 44.2 x 26 mm, 52 parts, among them J1 programmer, J2 USB_B_Micro, Q1 Q_PMOS_DSG, Q2 Q_NMOS_GSD, U1 ESP-WROOM-02, U2 RT8097AHGB, U3 RT8097AHGB, U4 NPIC6C596, U5 NPIC6C596

Commit message: Update to kicad6
Other:
- net class Default removed
